File: BMS-V1/BMS-V1.kicad_pcb (KiCad board)
At the start: 2 copper layers, 40 parts, among them J1 BATT+, J2 BATT-, J3 Conn_01x04_Pin, Q1 IQDH35N03LM5CG, Q2 IQDH35N03LM5CG

Commit message: Finished BMS
Parts:
- removed BMS1: ~, BMS_SPT:SOP65P640X120-20N
- removed R15: 10M, Resistor_SMD:R_0805_2012Metric_Pad1.20x1.40mm_HandSolder
- removed R16: 1M, Resistor_SMD:R_0805_2012Metric_Pad1.20x1.40mm_HandSolder
- removed R17: 3.3M, Resistor_SMD:R_0805_2012Metric_Pad1.20x1.40mm_HandSolder
- added C14: 0.1u, Capacitor_SMD:C_0805_2012Metric_Pad1.18x1.45mm_HandSolder, F.Cu at (118.4, 171.2)
- added C16: 1uF, Capacitor_SMD:C_0805_2012Metric_Pad1.18x1.45mm_HandSolder, F.Cu at (113.7, 148.6)
- added J4: Conn_01x05_Pin, Connector_PinHeader_2.54mm:PinHeader_1x05_P2.54mm_Vertical, F.Cu at (81.7, 174.5)
- added U1: BQ76920PW, Package_SO:TSSOP-20_4.4x6.5mm_P0.65mm, F.Cu at (111.4, 153.9)
- C1, C2, C3, C5: value 1u -> 0.1u
- C10, C11, C12, C13: value 0.1u -> 1uF
- C4, C6: value 1u -> 1uF
- C8: value 0.1u -> 4.7uF
- D1: value 100V -> 26V
- D2: value 16V -> 100V
- D3: value 26V -> 16V
- J1: value BATT+ -> Conn_01x04_Pin; footprint Connector_PinHeader_2.54mm:PinHeader_1x01_P2.54mm_Horizontal -> Connector_PinHeader_2.54mm:PinHeader_1x04_P2.54mm_Horizontal
- J2: value BATT- -> BATT+
- J3: value Conn_01x04_Pin -> BATT-; footprint Connector_PinHeader_2.54mm:PinHeader_1x04_P2.54mm_Horizontal -> Connector_PinHeader_2.54mm:PinHeader_1x01_P2.54mm_Horizontal
- Q1, Q2: footprint IDQH:IQDH35N03LM5ATMA1 -> Footprints:IFX-PG-TTFN-9-2-V
- R1: value 1k -> 10k; moved to B.Cu
- R10: value 470k -> 75
- R11: value 1k -> 75
- R12: value 100 -> 1M
- R13: value 1M -> 3.3M
- R14: value 100 -> 1k
- R2: value 10k -> 1k
- R3: value 75 -> 1k
- R4, R6: value 75 -> 100
- R5: value 75 -> 1M
- R7: value 1k -> 10M
- R8: value 10k -> 75
- R9: value 487k -> 75
- moved Q2 86.2 mm to (95.2, 178.8), turned to -90 degrees
- moved R13 83.7 mm to (109.9, 186.6)
- moved Q1 78.1 mm to (102.6, 178.7), turned to -90 degrees
- moved R7 74.6 mm to (109.2, 178.3)
- moved C13 67.5 mm to (92.3, 162.6)
- moved R12 65.8 mm to (109.9, 184.1), turned to 180 degrees
- moved C1 64.3 mm to (77.5, 141.6), turned to 180 degrees
- moved D2 64.2 mm to (94.2, 185.6)
- moved R8 62.9 mm to (96.3, 163.8), turned to 90 degrees
- moved R4 62.3 mm to (97.0, 171.7), turned to 90 degrees
- moved C7 62.0 mm to (102.6, 167.1)
- moved C2 62.0 mm to (77.5, 138.4)
- moved C12 60.4 mm to (99.7, 157.5), turned to 180 degrees
- moved C11 60.1 mm to (99.7, 153.9), turned to -90 degrees
- moved D3 59.7 mm to (110.9, 189.7), turned to 180 degrees
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Connections:
- C1 pad 1: GND -> Cell3
- C1 pad 2: Net-(BMS1-AVDD) -> Net-(C1-Pad2)
- C10 pad 1: Net-(Q1-SOURCE1) -> Net-(U1-VC3)
- C10 pad 2: Net-(C10-Pad2) -> Net-(U1-VC2)
- C11 pad 1: Net-(C10-Pad2) -> Net-(U1-VC2)
- C11 pad 2: GND -> Net-(U1-VC1)
- C12 pad 1: Cell3 -> Net-(U1-VC1)
- C12 pad 2: Net-(C12-Pad2) -> GND
- C13 pad 1: Net-(C12-Pad2) -> GND
- C13 pad 2: GND -> Net-(U1-VC0)
- C2 pad 1: Net-(BMS1-VDD) -> Net-(C1-Pad2)
- C3 pad 1: Net-(BMS1-VC3) -> SRN
- C3 pad 2: Net-(BMS1-VC2) -> GND
- C4 pad 1: Net-(BMS1-VC2) -> GND
- C4 pad 2: Net-(BMS1-VC1) -> Net-(U1-CAP1)
- C5 pad 1: Net-(BMS1-VC1) -> SRP
- C6 pad 2: Net-(BMS1-VC0) -> Net-(U1-REGSRC)
- C7 pad 1: SRN -> SRP
- C7 pad 2: GND -> SRN
- C8 pad 1: SRP -> GND
- C8 pad 2: SRN -> Net-(J4-Pin_1)
- C9 pad 1: SRP -> Net-(Q1-SOURCE1)
- C9 pad 2: GND -> Net-(C14-Pad1)
- D1 pad 1: Net-(D1-K) -> Cell3
- D1 pad 2: Net-(D1-A) -> GND
- D2 pad 1: Net-(D1-K) -> CHG
- D2 pad 2: GND -> Net-(D2-A)
- D3 pad 1: Cell3 -> CHG
- J2 pad 1: GND -> Cell3
- J3 pad 1: Cell3 -> GND
- Q1 pad 2: Net-(Q1-SOURCE1) -> Net-(Q1-DRAIN1)
- Q1 pad 9: Net-(Q1-GATE) -> DSG
- Q2 pad 2: GND -> Net-(Q1-DRAIN1)
- Q2 pad 9: Net-(D1-K) -> CHG
- R1 pad 1: Cell3 -> Net-(U1-VC1)
- R1 pad 2: Net-(BMS1-VDD) -> Net-(U1-TS1)
- R10 pad 1: GND -> Cell2
- R10 pad 2: Net-(BMS1-LD) -> Net-(U1-VC2)
- R11 pad 1: CHG -> Cell1
- R11 pad 2: Net-(BMS1-CHG) -> Net-(U1-VC1)
- R12 pad 1: GND -> CHG
- R12 pad 2: SRP -> Net-(D2-A)
- R13 pad 2: Net-(Q1-SOURCE1) -> CHG
- R14 pad 1: Net-(Q1-SOURCE1) -> Cell3
- R14 pad 2: SRN -> Net-(U1-BAT)
- R2 pad 1: Net-(BMS1-VDD) -> DSG
- R3 pad 1: Cell3 -> Net-(U1-CHG)
- R3 pad 2: Net-(BMS1-VC3) -> CHG
- R4 pad 1: Cell2 -> GND
- R4 pad 2: Net-(BMS1-VC2) -> SRP
- R5 pad 1: Cell1 -> GND
- R5 pad 2: Net-(BMS1-VC1) -> Net-(Q1-SOURCE1)
- R6 pad 1: GND -> Net-(Q1-SOURCE1)
- R6 pad 2: Net-(BMS1-VC0) -> SRN
- R7 pad 1: Net-(BMS1-DSG) -> Net-(Q1-SOURCE1)
- R8 pad 1: Net-(BMS1-VTB) -> GND
- R8 pad 2: Net-(BMS1-TS) -> Net-(U1-VC0)
- R9 pad 1: Net-(BMS1-OCDP) -> Cell3
- R9 pad 2: GND -> Net-(U1-VC3)
- TH1 pad 1: Net-(BMS1-TS) -> GND
- TH1 pad 2: GND -> Net-(U1-TS1)
Routing:
- net CHG: track 0.00 -> 72.6 mm
- net Net-(J4-Pin_1): track 0.00 -> 70.6 mm, vias 0 -> 1
- net Cell3: track 0.00 -> 49.2 mm
- net Net-(J4-Pin_2): track 0.00 -> 48.1 mm, vias 0 -> 1
- net Net-(J4-Pin_3): track 0.00 -> 42.4 mm, vias 0 -> 1
- net DSG: track 0.00 -> 34.0 mm
- net Net-(J4-Pin_4): track 0.00 -> 33.8 mm, vias 0 -> 1
- net Net-(U1-VC1): track 0.00 -> 30.8 mm, vias 0 -> 1
- net SRP: track 0.00 -> 23.7 mm
- net Net-(Q1-SOURCE1): track 0.00 -> 22.5 mm
- net SRN: track 0.00 -> 22.3 mm
- net GND: track 0.00 -> 22.0 mm, vias 0 -> 1
- net Net-(U1-VC0): track 0.00 -> 20.6 mm
- net Net-(U1-TS1): track 0.00 -> 16.6 mm
- net Net-(U1-VC2): track 0.00 -> 16.4 mm
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- added copper zone on B.Cu, net GND
- added copper zone on F.Cu, net GND
Other:
- board outline added: 62.4 x 62.2 mm
