File: BMS-V1/BMS-V1.kicad_sch (KiCad schematic)
At the start: 41 parts, among them J1 BATT+, J2 BATT-, J3 Conn_01x04_Pin, J4 Conn_01x05_Pin, Q1 IQDH35N03LM5CG, Q2 IQDH35N03LM5CG, U1 BQ76920PW

Commit message: Finished BMS
Parts:
- removed C21: 1uF, Capacitor_SMD:C_0805_2012Metric_Pad1.18x1.45mm_HandSolder, symbol Device:C_Small
- Q1, Q2: footprint IDQH:IQDH35N03LM5ATMA1 -> Footprints:IFX-PG-TTFN-9-2-V
- renumbered C12 to C1, C22 to C10, C23 to C11, C24 to C12, C25 to C13, C11 to C14, C20 to C16, C13 to C2, C7 to C3, C26 to C4, C9 to C5, C27 to C6, C8 to C7, C28 to C8, C10 to C9, D3 to D1, D1 to D2, D2 to D3, J3 to J1, J1 to J2, J2 to J3, R36 to R1, R33 to R10, R34 to R11, R16 to R12, R17 to R13, R29 to R14, R30 to R2, R31 to R3, R12 to R4, R13 to R5, R14 to R6, R15 to R7, R35 to R8, R32 to R9, TH4 to TH1
Connections:
- net CHG: now also D2.1 (K), D3.1 (K), Q2.9 (GATE), R12.1, R13.2
- net DSG: now also Q1.9 (GATE), R7.2
Other:
- moved on the sheet: C16, R14
