File: Final_design/BMS.kicad_sch (KiCad schematic)
At the start: 40 parts, among them J1 Conn_01x04_Pin, J3 BATT+, J4 BATT-, J5 Conn_01x05_Pin, Q5 IQDH35N03LM5CG, Q6 IQDH35N03LM5CG, U1 BQ76920PW

Commit message: Finished design, Must be reviewed
Parts:
- removed C18, C26: 0.1u, Capacitor_SMD:C_0805_2012Metric_Pad1.18x1.45mm_HandSolder, symbol Device:C_Small
- removed J5: Conn_01x05_Pin, Connector_PinHeader_2.54mm:PinHeader_1x05_P2.54mm_Vertical, symbol Connector:Conn_01x05_Pin
- added J5: Conn_01x04_Pin, Connector_PinHeader_2.54mm:PinHeader_1x04_P2.54mm_Vertical, symbol Connector:Conn_01x04_Pin
- added R28: 500k, Resistor_SMD:R_0805_2012Metric_Pad1.20x1.40mm_HandSolder, symbol Device:R_Small
- D1, D2, D3: footprint Diode_THT:D_DO-35_SOD27_P10.16mm_Horizontal -> Diode_SMD:D_SOD-123
- J1: footprint Connector_PinHeader_2.54mm:PinHeader_1x04_P2.54mm_Horizontal -> Connector_PinHeader_2.54mm:PinHeader_1x04_P2.54mm_Vertical
- J3, J4: footprint Connector_PinHeader_2.54mm:PinHeader_1x01_P2.54mm_Horizontal -> Connector_PinHeader_2.54mm:PinHeader_1x01_P2.54mm_Vertical
- R15: value 10M -> 1M
- R9: footprint Resistor_SMD:R_0805_2012Metric_Pad1.20x1.40mm_HandSolder -> Resistor_SMD:R_2512_6332Metric_Pad1.40x3.35mm_HandSolder
- TH1: footprint Connector_PinHeader_1.27mm:PinHeader_1x02_P1.27mm_Horizontal -> Resistor_SMD:R_0603_1608Metric_Pad0.98x0.95mm_HandSolder
Connections:
- net +BATT: now also U1.9 (REGSRC)
- net ALERT: now also J5.3 (Pin_3), R28.2
- net GND: now also J5.4 (Pin_4); no longer C12.2, C13.1, C14.2, C17.1, C22.2, C24.1, C25.2, D1.2 (A), J1.4 (Pin_4), R16.1, R8.1, R9.1, TH1.1, U1.3 (VSS)
- net SCL: now also J5.2 (Pin_2)
- net SDA: now also J5.1 (Pin_1)
- net -BATT: now reaches C15.2
- net -BATT: now also C12.2, C13.1, C14.2, C17.1, C22.2, C24.1, C25.2, D1.2 (A), J1.4 (Pin_4), R16.1, R8.1, R9.1, TH1.1, U1.3 (VSS), R28.1; no longer U1.9 (REGSRC)
- no-connect marks 1 -> 0
Other:
- note added: "MCU"
- moved on the sheet: C25, R16
