File: Final_design/Charger.kicad_sch (KiCad schematic)
At the start: 34 parts, among them J9 Conn_01x03_Pin, Q11 40V, 10A, Q7 60V, 115mA, Q8 40V, 10A, U6 BQ24650

Commit message: Finished design, Must be reviewed
Parts:
- removed D10: Not Decided, Package_TO_SOT_SMD:TO-277B, symbol Diode:Fuxinsemi_PDS760
- removed F3: Not Decided, symbol Device:Fuse_Small
- removed J9: Conn_01x03_Pin, Connector_PinHeader_2.54mm:PinHeader_1x03_P2.54mm_Vertical, symbol Connector:Conn_01x03_Pin
- added J13: Conn_01x02_Pin, TerminalBlock_Phoenix:TerminalBlock_Phoenix_MKDS-1,5-2_1x02_P5.00mm_Horizontal, symbol Connector:Conn_01x02_Pin
- added J15: Conn_01x04_Pin, Connector_PinHeader_2.54mm:PinHeader_1x04_P2.54mm_Vertical, symbol Connector:Conn_01x04_Pin
- added J2: Conn_01x02_Pin, Connector_PinSocket_2.54mm:PinSocket_1x02_P2.54mm_Vertical, symbol Connector:Conn_01x02_Pin
- added R46: 10k, Resistor_SMD:R_0805_2012Metric_Pad1.20x1.40mm_HandSolder, symbol Device:R_Small
- C32: footprint Capacitor_SMD:C_0603_1608Metric_Pad1.08x0.95mm_HandSolder -> Capacitor_SMD:C_0805_2012Metric_Pad1.18x1.45mm_HandSolder
- D5, D6: footprint Diode_SMD:D_0603_1608Metric -> LED_SMD:LED_0805_2012Metric_Pad1.15x1.40mm_HandSolder
- D9: footprint Package_TO_SOT_SMD:SOT-23 -> Package_TO_SOT_SMD:SOT-23_Handsoldering
- Q11, Q8: footprint Package_SO:PowerPAK_SO-8_Dual -> Package_TO_SOT_THT:TO-220-3_Vertical
- Q7: footprint Package_TO_SOT_SMD:SOT-23 -> Package_TO_SOT_THT:TO-220-3_Vertical
- TH2: footprint Resistor_SMD:R_0805_2012Metric_Pad1.20x1.40mm_HandSolder -> Resistor_SMD:R_0603_1608Metric_Pad0.98x0.95mm_HandSolder
Connections:
- net +BATT: now also J15.3 (Pin_3), J2.2 (Pin_2); no longer D4.2 (A), R32.1, R33.1
- net GND: now also J13.1 (Pin_1), J15.4 (Pin_4)
- net MPPSET: now also J15.2 (Pin_2), R46.1
- net at C30.2, C32.2, C34.2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: now also J2.1 (Pin_1)
- new net +3.3V: J15.1 (Pin_1), R46.2
- new net +SOLAR: D4.2 (A), J13.2 (Pin_2), R32.1, R33.1
Other:
- note added: "External Connectors"
- note added: "Q8 and Q11 will be changed"
- note added: "Tjek om Q7 gate må være gnd"
- note removed: "R3 Must be 1 W-rated part"
- moved on the sheet: C27, C28, C29, C30, C31, C32, C33, C34, C35, C36, D4, D5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
