File: Final_design/MCU.kicad_sch (KiCad schematic)
At the start: 17 parts, among them J10 Conn_01x03_Pin, J6 Conn_01x05_Pin, J7 Conn_01x10_Pin, J8 Conn_01x10_Pin, U2 L7805, U7 ATmega32A-P, Y1 8MHz

Commit message: Finished design, Must be reviewed
Parts:
- removed J10: Conn_01x03_Pin, Connector_PinHeader_2.54mm:PinHeader_1x03_P2.54mm_Vertical, symbol Connector:Conn_01x03_Pin
- removed J6: Conn_01x05_Pin, Connector_PinHeader_2.54mm:PinHeader_1x05_P2.54mm_Vertical, symbol Connector:Conn_01x05_Pin
- removed J7: Conn_01x10_Pin, Connector_PinSocket_2.54mm:PinSocket_1x10_P2.54mm_Vertical, symbol Connector:Conn_01x10_Pin
- removed U2: L7805, Package_TO_SOT_THT:TO-220-3_Vertical, symbol Regulator_Linear:L7805
- removed U7: ATmega32A-P, Package_DIP:DIP-40_W15.24mm, symbol MCU_Microchip_ATmega:ATmega32A-P
- added C41: 0.33uF, Capacitor_SMD:C_0805_2012Metric_Pad1.18x1.45mm_HandSolder, symbol Device:C_Small
- added C42: 10uF, Capacitor_SMD:C_1206_3216Metric_Pad1.33x1.80mm_HandSolder, symbol Device:C_Small
- added C47, C48, C49, C50: 0.1uf, Capacitor_SMD:C_0805_2012Metric_Pad1.18x1.45mm_HandSolder, symbol Device:C_Small
- added J12, J7: Conn_01x07_Pin, Connector_PinHeader_2.54mm:PinHeader_1x07_P2.54mm_Vertical, symbol Connector:Conn_01x07_Pin
- added J16, J6: Conn_01x04_Pin, Connector_PinHeader_2.54mm:PinHeader_1x04_P2.54mm_Vertical, symbol Connector:Conn_01x04_Pin
- added R44, R45: 4k7, Resistor_SMD:R_0805_2012Metric_Pad1.20x1.40mm_HandSolder, symbol Device:R_Small
- added R47, R48, R49: 1k, Resistor_SMD:R_0805_2012Metric_Pad1.20x1.40mm_HandSolder, symbol Device:R_Small
- added U10: ATmega32A-A, Package_QFP:TQFP-44_10x10mm_P0.8mm, symbol MCU_Microchip_ATmega:ATmega32A-A
- added U7: LM1117T-3.3, Package_TO_SOT_THT:TO-220-3_Vertical, symbol Regulator_Linear:LM1117T-3.3
- added U8: L7805, Package_TO_SOT_THT:TO-220-3_Vertical, symbol Regulator_Linear:L7805
- C19: footprint Capacitor_THT:C_Disc_D5.0mm_W2.5mm_P5.00mm -> Capacitor_SMD:C_0805_2012Metric_Pad1.18x1.45mm_HandSolder
- C23: value 0.1uF -> 10uF; footprint Capacitor_THT:C_Disc_D5.0mm_W2.5mm_P5.00mm -> Capacitor_SMD:C_1206_3216Metric_Pad1.33x1.80mm_HandSolder
- C37, C38, C39: footprint Capacitor_THT:C_Axial_L3.8mm_D2.6mm_P7.50mm_Horizontal -> Capacitor_SMD:C_0805_2012Metric_Pad1.18x1.45mm_HandSolder
- D11, D12: footprint Diode_SMD:D_0603_1608Metric -> LED_SMD:LED_0805_2012Metric_Pad1.15x1.40mm_HandSolder
- R41: footprint Resistor_THT:R_Axial_DIN0207_L6.3mm_D2.5mm_P10.16mm_Horizontal -> Resistor_SMD:R_0805_2012Metric_Pad1.20x1.40mm_HandSolder
Connections:
- net +5V: now also C42.1, J7.5 (Pin_5), U8.3 (OUT); no longer C23.1, C39.1, J8.2 (Pin_2), R41.1
- net +BATT: now also C41.1, J16.3 (Pin_3), J7.6 (Pin_6), U7.3 (VI), U8.1 (IN)
- net ALERT: now also J6.3 (Pin_3), U10.11 (PD2)
- net GND: now also C41.2, C42.2, C47.2, C48.2, C49.2, C50.2, J16.4 (Pin_4), J6.4 (Pin_4), J7.7 (Pin_7), U10.18 (GND), U10.28 (GND), U10.39 (GND), U10.6 (GND), U7.1 (GND), U8.2 (GND)
- net LED0: now also U10.37 (PA0)
- net LED1: now also U10.36 (PA1)
- net LIN1-PC2: now also J7.3 (Pin_3), U10.21 (PC2)
- net LIN2-PC3: now also J7.4 (Pin_4), U10.22 (PC3)
- net MISO: now also R49.2, U10.2 (PB6); no longer J8.9 (Pin_9)
- net MOSI: now also R47.2, U10.1 (PB5); no longer J8.1 (Pin_1)
- net MPPSET: now also J16.2 (Pin_2), U10.35 (PA2)
- net PWM1-PB3: now also J7.1 (Pin_1), U10.43 (PB3)
- net PWM2-PD5: now also J7.2 (Pin_2), U10.14 (PD5)
- net RESET: now also U10.4 (~{RESET})
- net SCK: now also R48.2, U10.3 (PB7); no longer J8.7 (Pin_7)
- net SCL: now also J6.2 (Pin_2), R45.2, U10.19 (PC0)
- net SDA: now also J6.1 (Pin_1), R44.2, U10.20 (PC1)
- net at C38.1, Y1.2: now also U10.7 (XTAL2)
- net at C37.1, Y1.1: now also U10.8 (XTAL1)
- new net: J8.7 (Pin_7), R48.1
- new net: J8.1 (Pin_1), R47.1
- new net: J8.9 (Pin_9), R49.1
- new net: C47.1, U10.29 (AREF)
- new net +3.3V: C23.1, C39.1, C48.1, C49.1, C50.1, J16.1 (Pin_1), J8.2 (Pin_2), R41.1, R44.1, R45.1, U10.17 (VCC), U10.27 (AVCC), U10.38 (VCC), U10.5 (VCC), U7.2 (VO)
- new net CLOCK: J12.3 (Pin_3), U10.32 (PA5)
- new net CONTROL: J12.5 (Pin_5), U10.30 (PA7)
- new net CW: J12.4 (Pin_4), U10.31 (PA6)
- new net ENABLE: J12.6 (Pin_6), U10.25 (PC6)
- new net HALF: J12.2 (Pin_2), U10.33 (PA4)
- new net HOME: J12.7 (Pin_7), U10.26 (PC7)
- new net RESET_STEP: J12.1 (Pin_1), U10.34 (PA3)
- no-connect marks 3 -> 12
Other:
- note added: "H_Bridge"
- note added: "I will ensure to turn off the battery before using the USB-connector"
- note added: "MOTOR - Connections"
- note added: "Stepper"
- note removed: "MCU - Connections"
- moved on the sheet: C37, C38, C39, D11, D12, J8, R41, R42, R43, Y1
