File: Final_design/Motor.kicad_sch (KiCad schematic)
At the start: 28 parts, among them J2 Conn_01x10_Pin, M1 Motor_DC, Q1 IRLZ34N, Q2 IRLZ34N, Q3 IRLZ34N, Q4 IRLZ34N, U3 IR2010, U4 IR2010

Commit message: Finished design, Must be reviewed
Parts:
- removed J2: Conn_01x10_Pin, Connector_PinSocket_2.54mm:PinSocket_1x10_P2.54mm_Vertical, symbol Connector:Conn_01x10_Pin
- added C43: 3.3nF, Capacitor_SMD:C_0805_2012Metric_Pad1.18x1.45mm_HandSolder, symbol Device:C_Small
- added C44, C45, C46: 100nF, Capacitor_SMD:C_0805_2012Metric_Pad1.18x1.45mm_HandSolder, symbol Device:C_Small
- added D10, D13, D14, D15, D16, D17, D18, D19: D_Schottky_Small_Filled, Diode_SMD:D_SMA_Handsoldering, symbol Device:D_Schottky_Small_Filled
- added J11, J14: Conn_01x07_Pin, Connector_PinHeader_2.54mm:PinHeader_1x07_P2.54mm_Vertical, symbol Connector:Conn_01x07_Pin
- added M2: Stepper_Motor_bipolar, TerminalBlock_Phoenix:TerminalBlock_Phoenix_MKDS-1,5-4_1x04_P5.00mm_Horizontal, symbol Motor:Stepper_Motor_bipolar
- added R10: 22k, Resistor_SMD:R_0805_2012Metric_Pad1.20x1.40mm_HandSolder, symbol Device:R_Small
- added R11, R12: 0.5, Resistor_SMD:R_0805_2012Metric_Pad1.20x1.40mm_HandSolder, symbol Device:R_Small
- added R13: 39k, Resistor_SMD:R_0805_2012Metric_Pad1.20x1.40mm_HandSolder, symbol Device:R_Small
- added R21, R22: 10k, Resistor_SMD:R_0805_2012Metric_Pad1.20x1.40mm_HandSolder, symbol Device:R_Small
- added U2: L297, Package_DIP:CERDIP-20_W7.62mm_SideBrazed, symbol Driver_Motor:L297
- added U5: L298N, Package_TO_SOT_THT:TO-220-15_P2.54x5.08mm_StaggerOdd_Lead4.58mm_Vertical, symbol Driver_Motor:L298N
- C10, C11, C6, C7: footprint Capacitor_THT:C_Disc_D5.0mm_W2.5mm_P5.00mm -> Capacitor_SMD:C_0805_2012Metric_Pad1.18x1.45mm_HandSolder
- C4, C5: footprint Capacitor_THT:CP_Radial_D5.0mm_P2.00mm -> Capacitor_SMD:C_1210_3225Metric_Pad1.33x2.70mm_HandSolder
- C8, C9: footprint Capacitor_THT:CP_Radial_D5.0mm_P2.00mm -> Capacitor_SMD:C_0805_2012Metric_Pad1.18x1.45mm_HandSolder
- D7, D8: footprint Diode_THT:D_DO-35_SOD27_P7.62mm_Horizontal -> Diode_SMD:D_SOD-523
- R18, R19, R2, R20, R23, R3, R4, R5: footprint Resistor_THT:R_Axial_DIN0207_L6.3mm_D2.5mm_P10.16mm_Horizontal -> Resistor_SMD:R_0805_2012Metric_Pad1.20x1.40mm_HandSolder
Connections:
- net LIN1-PC0 is gone; now on net LIN1-PC2: U3.12 (LIN)
- net LIN2-PC1 is gone; now on net LIN2-PC3: U4.12 (LIN)
- net MOTOR_IN1 is gone; now on net PWM1-PB3: U3.10 (HIN)
- net MOTOR_IN2 is gone; now on net PWM2-PD5: U4.10 (HIN)
- net +5V: now also C44.1, C46.1, J14.5 (Pin_5), R10.1, R13.1, U2.12 (Vs), U5.9 (Vss)
- net +BATT: now also D10.1 (K), D13.1 (K), D14.1 (K), D15.1 (K), J14.6 (Pin_6), U5.4 (Vs)
- net GND: now also C43.2, C44.2, C45.2, C46.2, D16.2 (A), D17.2 (A), D18.2 (A), D19.2 (A), J14.7 (Pin_7), R11.2, R12.2, R21.2, R22.2, U2.2 (GND), U5.8 (GND)
- net LIN1-PC2: now also J14.3 (Pin_3)
- net LIN2-PC3: now also J14.4 (Pin_4)
- net PWM1-PB3: now also J14.1 (Pin_1)
- net PWM2-PD5: now also J14.2 (Pin_2)
- new net: D13.2 (A), D17.1 (K), M2.2 (-), U5.3 (OUT2)
- new net: R12.1, U2.13 (SENS2), U5.15 (SENSE_B)
- new net: R11.1, U2.14 (SENS1), U5.1 (SENSE_A)
- new net: C45.1, R13.2, R21.1, U2.15 (Vref)
- new net: C43.1, R10.2, U2.16 (OSC)
- new net: U2.4 (A), U5.5 (IN1)
- new net: U2.5 (INH1), U5.6 (EnA)
- new net: U2.6 (B), U5.7 (IN2)
- new net: U2.7 (C), U5.10 (IN3)
- new net: U2.8 (INH2), U5.11 (EnB)
- new net: U2.9 (D), U5.12 (IN4)
- new net: D15.2 (A), D19.1 (K), M2.4, U5.14 (OUT4)
- new net: D10.2 (A), D16.1 (K), M2.1, U5.2 (OUT1)
- new net: D14.2 (A), D18.1 (K), M2.3, U5.13 (OUT3)
- new net CLOCK: J11.3 (Pin_3), U2.18 (CLOCK)
- new net CONTROL: J11.5 (Pin_5), U2.11 (CONTROL)
- new net CW: J11.4 (Pin_4), U2.17 (CW)
- new net ENABLE: J11.6 (Pin_6), R22.1, U2.10 (ENABLE)
- new net HALF: J11.2 (Pin_2), U2.19 (HALF)
- new net HOME: J11.7 (Pin_7), U2.3 (HOME)
- new net RESET_STEP: J11.1 (Pin_1), U2.20 (RESET)
Other:
- note added: "5 A / 40-60 V"
- note added: "H-Bridge"
- note added: "Must be changed as IR2010 requires 10V min"
- note added: "Stepper"
- note added: "Stepper Motor"
- moved on the sheet: C1, C40, M1, Q1, Q2, Q3, Q4, R18, R19, R2, R20, R23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
